File: USB-Charger/Untitled.kicad_pcb (KiCad board)
At the start: 2 copper layers, 25.4 x 50.8 mm, 18 parts, among them J1 73725-0110BLF, U1 conv

Commit message: update projects
Routing:
- net GND: vias 3 -> 6
- net (no net): vias 0 -> 2
Changed lines of the file:
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@@
     (thickness 1.6)
     (drawings 4)
-    (tracks 206)
+    (tracks 211)
     (zones 0)
     (modules 18)
@@
     (45 Margin user)
     (46 B.CrtYd user)
-    (47 F.CrtYd user)
+    (47 F.CrtYd user hide)
     (48 B.Fab user)
-    (49 F.Fab user)
+    (49 F.Fab user hide)
   )
   (setup
@@
   (gr_line (start 128.27 139.7) (end 153.67 139.7) (layer Edge.Cuts) (width 0.15))
   (gr_line (start 128.27 88.9) (end 128.27 139.7) (layer Edge.Cuts) (width 0.15))
+  (via (at 153.035 89.789) (size 0.8) (drill 0.4) (layers F.Cu B.Cu) (net 0))
+  (via (at 142.113 127.8255) (size 0.8) (drill 0.4) (layers F.Cu B.Cu) (net 0))
   (via (at 145.288 122.809) (size 0.8) (drill 0.4) (layers F.Cu B.Cu) (net 1))
   (segment (start 146.746 123.825) (end 146.304 123.825) (width 0.25) (layer F.Cu) (net 1))
@@
   (segment (start 141.732 105.217) (end 143.129 106.614) (width 0.635) (layer F.Cu) (net 3))
   (segment (start 141.732 105.029) (end 141.732 105.217) (width 0.635) (layer F.Cu) (net 3))
+  (via (at 130.937 89.9795) (size 0.8) (drill 0.4) (layers F.Cu B.Cu) (net 3))
+  (via (at 129.8575 137.922) (size 0.8) (drill 0.4) (layers F.Cu B.Cu) (net 3))
+  (via (at 152.4 138.43) (size 0.8) (drill 0.4) (layers F.Cu B.Cu) (net 3))
   (segment (start 143.256 119.307) (end 143.256 118.557) (width 0.25) (layer F.Cu) (net 4))
   (segment (start 143.546 119.597) (end 143.256 119.307) (width 0.25) (layer F.Cu) (net 4))
