File: wireless_proj/wireless_proj.sch (KiCad schematic (older format))
At the start: 19 parts

Commit message: lalala
Parts:
- removed M?: MNMOS, symbol pspice:MNMOS
- added M1: Q_NMOS_DGS, Package_TO_SOT_THT:TO-3P-3_Horizontal_TabDown, symbol Device:Q_NMOS_DGS
- C1, C2: renamed from C?; value C -> 10u; footprint (none) -> Capacitor_SMD:C_1812_4532Metric_Pad1.30x3.40mm_HandSolder
- D1: renamed from D?; footprint (none) -> Diode_SMD:D_2512_6332Metric_Pad1.52x3.35mm_HandSolder
- D2: renamed from D?; footprint (none) -> Diode_SMD:D_3220_8050Metric_Pad2.65x5.15mm_HandSolder
- J1, P_in1: renamed from J?; footprint (none) -> Connector_PinHeader_2.54mm:PinHeader_1x02_P2.54mm_Horizontal
- J2, J3: renamed from J?; footprint (none) -> Connector_PinHeader_2.54mm:PinHeader_1x01_P2.54mm_Horizontal
- J4: renamed from J?; footprint (none) -> Connector_PinHeader_2.54mm:PinHeader_1x02_P2.54mm_Vertical
- LED1: renamed from D?; footprint (none) -> LED_THT:LED_D5.0mm
- R1: renamed from R?; value R -> 1; footprint (none) -> Resistor_SMD:R_2010_5025Metric_Pad1.52x2.65mm_HandSolder
- R2, R3: renamed from R?; value R -> 200; footprint (none) -> Resistor_SMD:R_2010_5025Metric_Pad1.52x2.65mm_HandSolder
- R4: renamed from R?; value R -> 4.99k; footprint (none) -> Resistor_SMD:R_2010_5025Metric_Pad1.52x2.65mm_HandSolder
- Rl1: renamed from Rl; value R -> 200; footprint (none) -> Resistor_SMD:R_2010_5025Metric_Pad1.52x2.65mm_HandSolder
- TH1: renamed from TH?; footprint (none) -> Resistor_SMD:R_2010_5025Metric_Pad1.52x2.65mm_HandSolder
- U1: renamed from U?; footprint Package_TO_SOT_SMD:SOT-23-5 -> Package_TO_SOT_SMD:SOT-23-8
- U2: renamed from U?; footprint digikey-footprints:TO-220-3 -> Connector:FanPinHeader_1x03_P2.54mm_Vertical
Connections:
- net labels added: GNDPWR
- wire segments 39 -> 42
